Commit message: imu joint is fixed

File: urdf/turtlebot3_waffle_pi.urdf.xacro (robot description, xacro)
@@ -130,7 +130,5 @@
     </inertial>
   </link>
-  <joint name="imu_joint" type="revolute">
-    <axis xyz="0 0 1"/>
-    <limit effort="1000.0" lower="0.0" upper="0" velocity="0"/>
+  <joint name="imu_joint" type="fixed">
     <parent link="$(arg prefix)base_link"/>
     <child link="$(arg prefix)imu_link"/>
