Commit message: cam ok / imu has wrong frame

File: urdf/turtlebot3_gazebo.xacro (robot description, xacro)
@@ -9,124 +9,58 @@
  <xacro:arg name="odom_topic"    default="odom"/>
  <xacro:arg name="publish_odom"    default="false"/>
-  <gazebo reference="$(arg prefix)base_link">
-    <material>Gazebo/DarkGrey</material>
-  </gazebo>
-  <gazebo reference="$(arg prefix)wheel_left_link">
-    <mu1>0.1</mu1>
-    <mu2>0.1</mu2>
-    <kp>500000.0</kp>
-    <kd>10.0</kd>
-    <minDepth>0.001</minDepth>
-    <maxVel>0.1</maxVel>
-    <fdir1>1 0 0</fdir1>
-    <material>Gazebo/FlatBlack</material>
-  </gazebo>
-  <gazebo reference="$(arg prefix)wheel_right_link">
-    <mu1>0.1</mu1>
-    <mu2>0.1</mu2>
-    <kp>500000.0</kp>
-    <kd>10.0</kd>
-    <minDepth>0.001</minDepth>
-    <maxVel>0.1</maxVel>
-    <fdir1>1 0 0</fdir1>
-    <material>Gazebo/FlatBlack</material>
-  </gazebo>
-  <gazebo reference="$(arg prefix)caster_back_right_link">
-    <mu1>0.1</mu1>
-    <mu2>0.1</mu2>
-    <kp>1000000.0</kp>
-    <kd>100.0</kd>
-    <minDepth>0.001</minDepth>
-    <maxVel>1.0</maxVel>
-    <material>Gazebo/FlatBlack</material>
-  </gazebo>
-  <gazebo reference="$(arg prefix)caster_back_left_link">
-    <mu1>0.1</mu1>
-    <mu2>0.1</mu2>
-    <kp>1000000.0</kp>
-    <kd>100.0</kd>
-    <minDepth>0.001</minDepth>
-    <maxVel>1.0</maxVel>
-    <material>Gazebo/FlatBlack</material>
-  </gazebo>
-  <gazebo reference="$(arg prefix)imu_link">
-    <sensor name="tb3_imu" type="imu">
-        <always_on>true</always_on>
-        <visualize>$(arg imu_visual)</visualize>
-        <update_rate>50</update_rate>
-        <imu>
-          <angular_velocity>
-            <x>
-              <noise type="gaussian">
-                <mean>0.0</mean>
-                <stddev>2e-4</stddev>
-              </noise>
-            </x>
-            <y>
-              <noise type="gaussian">
-                <mean>0.0</mean>
-                <stddev>2e-4</stddev>
-              </noise>
-            </y>
-            <z>
-              <noise type="gaussian">
-                <mean>0.0</mean>
-                <stddev>2e-4</stddev>
-              </noise>
-            </z>
-          </angular_velocity>
-          <linear_acceleration>
-            <x>
-              <noise type="gaussian">
-                <mean>0.0</mean>
-                <stddev>1.7e-2</stddev>
-              </noise>
-            </x>
-            <y>
-              <noise type="gaussian">
-                <mean>0.0</mean>
-                <stddev>1.7e-2</stddev>
-              </noise>
-            </y>
-            <z>
-              <noise type="gaussian">
-                <mean>0.0</mean>
-                <stddev>1.7e-2</stddev>
-              </noise>
-            </z>
-          </linear_acceleration>
-        </imu>
-        <plugin name="turtlebot3_imu" filename="libgazebo_ros_imu_sensor.so">
-          <ros>
-            <remapping>~/out:=imu</remapping>
-          </ros>
-        </plugin>
-    </sensor>
-    <material>Gazebo/Grey</material>
-  </gazebo>
+<gazebo reference="$(arg prefix)base_link">
+  <material>Gazebo/DarkGrey</material>
+</gazebo>
+<gazebo reference="$(arg prefix)wheel_left_link">
+  <mu1>0.1</mu1>
+  <mu2>0.1</mu2>
+  <kp>500000.0</kp>
+  <kd>10.0</kd>
+  <minDepth>0.001</minDepth>
+  <maxVel>0.1</maxVel>
+  <fdir1>1 0 0</fdir1>
+  <material>Gazebo/FlatBlack</material>
+</gazebo>
+<gazebo reference="$(arg prefix)wheel_right_link">
+  <mu1>0.1</mu1>
+  <mu2>0.1</mu2>
+  <kp>500000.0</kp>
+  <kd>10.0</kd>
+  <minDepth>0.001</minDepth>
+  <maxVel>0.1</maxVel>
+  <fdir1>1 0 0</fdir1>
+  <material>Gazebo/FlatBlack</material>
+</gazebo>
+<gazebo reference="$(arg prefix)caster_back_right_link">
+  <mu1>0.1</mu1>
+  <mu2>0.1</mu2>
+  <kp>1000000.0</kp>
+  <kd>100.0</kd>
+  <minDepth>0.001</minDepth>
+  <maxVel>1.0</maxVel>
+  <material>Gazebo/FlatBlack</material>
+</gazebo>
+<gazebo reference="$(arg prefix)caster_back_left_link">
+  <mu1>0.1</mu1>
+  <mu2>0.1</mu2>
+  <kp>1000000.0</kp>
+  <kd>100.0</kd>
+  <minDepth>0.001</minDepth>
+  <maxVel>1.0</maxVel>
+  <material>Gazebo/FlatBlack</material>
+</gazebo>
+<gazebo reference="$(arg prefix)imu_link">
+<sensor name="imu_link" type="imu">
+    <imu_frame_id>$(arg prefix)imu_link</imu_frame_id>
+    <always_on>1</always_on>
+    <update_rate>1</update_rate>
+<!--     <visualize>true</viualize> -->
+    <topic>$(arg prefix)imu</topic>
+</sensor>
+</gazebo>
  <gazebo>
-    <!-- classic -->
-    <plugin name="turtlebot3_diff_drive" filename="libgazebo_ros_diff_drive.so">
-      <ros>
-        <remapping>odom:=$(arg odom_topic)</remapping>
-        <remapping>cmd_vel:=$(arg cmd_vel_topic)</remapping>
-      </ros>
-      <update_rate>30</update_rate>
-      <left_joint>wheel_left_joint</left_joint>
-      <right_joint>wheel_right_joint</right_joint>
-      <wheel_separation>${wheel_separation}</wheel_separation>
-      <wheel_diameter>0.066</wheel_diameter>
-      <max_wheel_torque>20</max_wheel_torque>
-      <max_wheel_acceleration>1.0</max_wheel_acceleration>
-      <publish_odom>$(arg publish_odom)</publish_odom>
-      <publish_odom_tf>true</publish_odom_tf>
-      <publish_wheel_tf>false</publish_wheel_tf>
-      <odometry_frame>$(arg prefix)odom</odometry_frame>
-      <robot_base_frame>$(arg prefix)base_footprint</robot_base_frame>
-    </plugin>
-    <!-- Ignition -->
     <plugin
-      filename="libignition-gazebo-diff-drive-system.so"
-      name="ignition::gazebo::systems::DiffDrive">
+      filename="libgz-sim-diff-drive-system.so"
+      name="gz::sim::systems::DiffDrive">
       <left_joint>wheel_left_joint</left_joint>
       <right_joint>wheel_right_joint</right_joint>
@@ -138,6 +72,7 @@
   <gazebo reference="$(arg prefix)base_scan">
     <material>Gazebo/FlatBlack</material>
-    <sensor type="ray" name="lds_lfcd_sensor">
+    <sensor type="lidar" name="lds_lfcd_sensor">
       <pose>0 0 0 0 0 0</pose>
+      <topic>$(arg prefix)scan</topic>
       <visualize>$(arg laser_visual)</visualize>
       <update_rate>5</update_rate>
@@ -162,11 +97,4 @@
         </noise>
       </ray>
-    <plugin name="scan" filename="libgazebo_ros_ray_sensor.so">
-      <ros>
-        <remapping>~/out:=scan</remapping>
-      </ros>
-      <output_type>sensor_msgs/LaserScan</output_type>
-      <frame_name>$(arg prefix)base_scan</frame_name>
-    </plugin>
     </sensor>
   </gazebo>
@@ -174,47 +102,27 @@
   <xacro:if value="$(arg use_cam)">
   <gazebo reference="$(arg prefix)camera_rgb_frame">
-    <sensor type="camera" name="pi_camera">
-      <always_on>true</always_on>
-      <visualize>$(arg camera_visual)</visualize>
-      <camera>
-          <horizontal_fov>1.085595</horizontal_fov>
-          <image>
-              <width>640</width>
-              <height>480</height>
-              <format>R8G8B8</format>
-          </image>
-          <clip>
-              <near>0.03</near>
-              <far>100</far>
-          </clip>
-      </camera>
-      <plugin name="camera_controller" filename="libgazebo_ros_camera.so">
-        <alwaysOn>true</alwaysOn>
-        <updateRate>30.0</updateRate>
-        <hackBaseline>0.07</hackBaseline>
-        <distortionK1>0.0</distortionK1>
-        <distortionK2>0.0</distortionK2>
-        <distortionK3>0.0</distortionK3>
-        <distortionT1>0.0</distortionT1>
-        <distortionT2>0.0</distortionT2>
-        <plugin name="camera_driver" filename="libgazebo_ros_camera.so">
-            <frame_name>$(arg prefix)camera_rgb_frame</frame_name>
-          </plugin>
-      </plugin>
-    </sensor>
+    <sensor name="camera" type="camera">
+    <camera>
+    <optical_frame_id>$(arg prefix)camera_rgb_optical_frame</optical_frame_id>
+    <horizontal_fov>1.047</horizontal_fov>
+    <image>
+        <width>640</width>
+        <height>400</height>
+    </image>
+    <clip>
+        <near>0.3</near>
+        <far>100</far>
+    </clip>
+    </camera>
+    <always_on>1</always_on>
+    <update_rate>30</update_rate>
+    <visualize>true</visualize>
+    <topic>$(arg prefix)image</topic>
+    <enable_metrics>false</enable_metrics>
+</sensor>
   </gazebo>
 </xacro:if>
    <gazebo>
-        <!-- classic -->
-      <plugin name="turtlebot3_joint_state" filename="libgazebo_ros_joint_state_publisher.so">
-      <ros>
-        <!-- <namespace>/tb3</namespace> -->
-        <remapping>~/out:=joint_states</remapping>
-      </ros>
-      <update_rate>30</update_rate>
-      <joint_name>wheel_left_joint</joint_name>
-      <joint_name>wheel_right_joint</joint_name>
-    </plugin>
-      <plugin filename="libignition-gazebo-joint-state-publisher-system.so" name="ignition::gazebo::systems::JointStatePublisher"/>
+      <plugin filename="libgz-sim-joint-state-publisher-system.so" name="gz::sim::systems::JointStatePublisher"/>
     </gazebo>
 </robot>

Commit message: setup bringup

File: urdf/turtlebot3_gazebo.xacro (robot description, xacro)
@@ -51,10 +51,9 @@
 </gazebo>
 <gazebo reference="$(arg prefix)imu_link">
-<sensor name="imu_link" type="imu">
-    <imu_frame_id>$(arg prefix)imu_link</imu_frame_id>
+<sensor name="imu_sensor" type="imu">
     <always_on>1</always_on>
-    <update_rate>1</update_rate>
-<!--     <visualize>true</viualize> -->
+    <update_rate>20</update_rate>
     <topic>$(arg prefix)imu</topic>
+    <gz_frame_id>$(arg prefix)imu_link</gz_frame_id>
 </sensor>
 </gazebo>
@@ -72,7 +71,8 @@
   <gazebo reference="$(arg prefix)base_scan">
     <material>Gazebo/FlatBlack</material>
-    <sensor type="lidar" name="lds_lfcd_sensor">
-      <pose>0 0 0 0 0 0</pose>
+    <sensor type="gpu_ray" name="lds_lfcd_sensor">
+<!--       <pose>0 0 0 0 0 0</pose> -->
       <topic>$(arg prefix)scan</topic>
+      <gz_frame_id>$(arg prefix)base_scan</gz_frame_id>
       <visualize>$(arg laser_visual)</visualize>
       <update_rate>5</update_rate>

File: urdf/turtlebot3_waffle_pi.urdf.xacro (robot description, xacro)
@@ -130,10 +130,17 @@
     </inertial>
   </link>
-  <joint name="imu_joint" type="fixed">
+  <joint name="imu_joint" type="revolute">
+    <axis xyz="0 0 1"/>
+    <limit effort="1000.0" lower="0.0" upper="0" velocity="0"/>
     <parent link="$(arg prefix)base_link"/>
     <child link="$(arg prefix)imu_link"/>
     <origin xyz="0.0 0 0.068" rpy="0 0 0"/>
   </joint>
-  <link name="$(arg prefix)imu_link"/>
+  <link name="$(arg prefix)imu_link">
+        <inertial>
+      <mass value="0.001"/>
+      <inertia ixx="0.00000542" ixy="0.0" ixz="0.0" iyy="0.00002104" iyz="0.0" izz="0.00002604"/>
+    </inertial>
+  </link>
   <joint name="scan_joint" type="fixed">
     <parent link="$(arg prefix)base_link"/>

Commit message: much better Gz behavior through surface tags

File: urdf/turtlebot3_gazebo.xacro (robot description, xacro)
@@ -10,39 +10,13 @@
 </gazebo>
 <gazebo reference="$(arg prefix)wheel_left_link">
-  <mu1>0.1</mu1>
-  <mu2>0.1</mu2>
-  <kp>500000.0</kp>
-  <kd>10.0</kd>
-  <minDepth>0.001</minDepth>
-  <maxVel>0.1</maxVel>
-  <fdir1>1 0 0</fdir1>
   <material>Gazebo/FlatBlack</material>
 </gazebo>
 <gazebo reference="$(arg prefix)wheel_right_link">
-  <mu1>0.1</mu1>
-  <mu2>0.1</mu2>
-  <kp>500000.0</kp>
-  <kd>10.0</kd>
-  <minDepth>0.001</minDepth>
-  <maxVel>0.1</maxVel>
-  <fdir1>1 0 0</fdir1>
   <material>Gazebo/FlatBlack</material>
 </gazebo>
 <gazebo reference="$(arg prefix)caster_back_right_link">
-  <mu1>0.1</mu1>
-  <mu2>0.1</mu2>
-  <kp>1000000.0</kp>
-  <kd>100.0</kd>
-  <minDepth>0.001</minDepth>
-  <maxVel>1.0</maxVel>
   <material>Gazebo/FlatBlack</material>
 </gazebo>
 <gazebo reference="$(arg prefix)caster_back_left_link">
-  <mu1>0.1</mu1>
-  <mu2>0.1</mu2>
-  <kp>1000000.0</kp>
-  <kd>100.0</kd>
-  <minDepth>0.001</minDepth>
-  <maxVel>1.0</maxVel>
   <material>Gazebo/FlatBlack</material>
 </gazebo>

File: urdf/turtlebot3_waffle_pi.urdf.xacro (robot description, xacro)
@@ -26,5 +26,4 @@
     </collision>
     <inertial>
-      <origin xyz="0 0 0" rpy="0 0 0"/>
       <mass value="1.3729096e+00"/>
       <inertia ixx="8.7002718e-03" ixy="-4.7576583e-05" ixz="1.1160499e-04"
@@ -38,4 +37,5 @@
     <origin xyz="0.0 0.144 0.023" rpy="-1.57 0 0"/>
     <axis xyz="0 0 1"/>
+    <limit velocity="7.88" effort="10"/>
   </joint>
   <link name="$(arg prefix)wheel_left_link">
@@ -48,8 +48,15 @@
     </visual>
     <collision>
-      <origin xyz="0 0 0" rpy="0 0 0"/>
       <geometry>
         <cylinder length="0.018" radius="0.033"/>
       </geometry>
+            <surface>
+          <friction>
+              <ode>
+                  <mu>1</mu>
+                  <mu2>0</mu2>
+              </ode>
+          </friction>
+      </surface>
     </collision>
     <inertial>
@@ -66,4 +73,5 @@
     <origin xyz="0.0 -0.144 0.023" rpy="-1.57 0 0"/>
     <axis xyz="0 0 1"/>
+    <limit velocity="7.88" effort="10"/>
   </joint>
   <link name="$(arg prefix)wheel_right_link">
@@ -76,8 +84,15 @@
     </visual>
     <collision>
-      <origin xyz="0 0 0" rpy="0 0 0"/>
       <geometry>
         <cylinder length="0.018" radius="0.033"/>
       </geometry>
+        <surface>
+            <friction>
+                <ode>
+                    <mu>1</mu>
+                    <mu2>0</mu2>
+                </ode>
+            </friction>
+        </surface>
     </collision>
     <inertial>
@@ -98,6 +113,15 @@
       <origin xyz="0 0.001 0" rpy="0 0 0"/>
       <geometry>
-        <box size="0.030 0.009 0.020"/>
-      </geometry>
+<!--         <box size="0.030 0.009 0.020"/> -->
+        <sphere radius="0.009"/>
+      </geometry>
+        <surface>
+            <friction>
+                <ode>
+                    <mu>0</mu>
+                    <mu2>0</mu2>
+                </ode>
+            </friction>
+        </surface>
     </collision>
     <inertial>
@@ -118,6 +142,15 @@
       <origin xyz="0 0.001 0" rpy="0 0 0"/>
       <geometry>
-        <box size="0.030 0.009 0.020"/>
-      </geometry>
+<!--         <box size="0.030 0.009 0.020"/> -->
+        <sphere radius="0.009"/>
+      </geometry>
+      <surface>
+      <friction>
+          <ode>
+              <mu>0</mu>
+              <mu2>0</mu2>
+          </ode>
+      </friction>
+  </surface>
     </collision>
     <inertial>
