Commit message: adapt mesh definition to using Gazebo or the real robot

File: urdf/common_properties.xacro (robot description, xacro)
@@ -32,3 +32,15 @@
     <color rgba="1.0 1.0 1.0 1.0"/>
   </material>
+ <xacro:arg name="gazebo" default="false"/>
+ <xacro:if value="$(arg gazebo)">
+   <xacro:include filename="$(find turtlebot3_xacro)/urdf/turtlebot3_gazebo.xacro"/>
+ </xacro:if>
+ <xacro:macro name="mesh" params="mesh">
+   <xacro:if value="$(arg gazebo)">
+     <mesh filename="file://$(find turtlebot3_description)/meshes/${mesh}" scale="0.001 0.001 0.001"/>
+   </xacro:if>
+   <xacro:unless value="$(arg gazebo)">
+     <mesh filename="package://turtlebot3_description/meshes/${mesh}" scale="0.001 0.001 0.001"/>
+   </xacro:unless>
+ </xacro:macro>
 </robot>

File: urdf/turtlebot3_burger.urdf.xacro (robot description, xacro)
@@ -5,5 +5,4 @@
  <xacro:arg name="use_cam" default="false"/>
   <xacro:include filename="$(find turtlebot3_xacro)/urdf/common_properties.xacro"/>
-  <xacro:include filename="$(find turtlebot3_xacro)/urdf/turtlebot3_gazebo.xacro"/>
   <link name="$(arg prefix)base_footprint"/>
   <joint name="base_joint" type="fixed">
@@ -16,5 +15,5 @@
       <origin xyz="-0.032 0 0.0" rpy="0 0 0"/>
       <geometry>
-        <mesh filename="file://$(find turtlebot3_description)/meshes/bases/burger_base.stl" scale="0.001 0.001 0.001"/>
+        <xacro:mesh mesh="bases/burger_base.stl"/>
       </geometry>
       <material name="light_black"/>
@@ -44,5 +43,5 @@
       <origin xyz="0 0 0" rpy="1.57 0 0"/>
       <geometry>
-        <mesh filename="file://$(find turtlebot3_description)/meshes/wheels/left_tire.stl" scale="0.001 0.001 0.001"/>
+        <xacro:mesh mesh="wheels/left_tire.stl"/>
       </geometry>
       <material name="dark"/>
@@ -72,5 +71,5 @@
       <origin xyz="0 0 0" rpy="1.57 0 0"/>
       <geometry>
-        <mesh filename="file://$(find turtlebot3_description)/meshes/wheels/right_tire.stl" scale="0.001 0.001 0.001"/>
+        <xacro:mesh mesh="wheels/right_tire.stl"/>
       </geometry>
       <material name="dark"/>
@@ -125,5 +124,5 @@
       <origin xyz="0 0 0.0" rpy="0 0 0"/>
       <geometry>
-        <mesh filename="file://$(find turtlebot3_description)/meshes/sensors/lds.stl" scale="0.001 0.001 0.001"/>
+        <xacro:mesh mesh="sensors/lds.stl"/>
       </geometry>
       <material name="dark"/>

File: urdf/turtlebot3_waffle_pi.urdf.xacro (robot description, xacro)
@@ -5,6 +5,5 @@
  <xacro:arg name="use_cam"    default="true"/>
  <xacro:include filename="$(find turtlebot3_xacro)/urdf/common_properties.urdf"/>
- <xacro:include filename="$(find turtlebot3_xacro)/urdf/turtlebot3_gazebo.xacro"/>
-  <link name="$(arg prefix)base_footprint"/>
+ <link name="$(arg prefix)base_footprint"/>
   <joint name="base_joint" type="fixed">
     <parent link="$(arg prefix)base_footprint"/>
@@ -16,5 +15,5 @@
       <origin xyz="-0.064 0 0.0" rpy="0 0 0"/>
       <geometry>
-        <mesh filename="file://$(find turtlebot3_description)/meshes/bases/waffle_pi_base.stl" scale="0.001 0.001 0.001"/>
+        <xacro:mesh mesh="bases/waffle_pi_base.stl"/>
       </geometry>
       <material name="light_black"/>
@@ -44,5 +43,5 @@
       <origin xyz="0 0 0" rpy="1.57 0 0"/>
       <geometry>
-        <mesh filename="file://$(find turtlebot3_description)/meshes/wheels/left_tire.stl" scale="0.001 0.001 0.001"/>
+        <xacro:mesh mesh="wheels/left_tire.stl"/>
       </geometry>
       <material name="dark"/>
@@ -72,5 +71,5 @@
       <origin xyz="0 0 0" rpy="1.57 0 0"/>
       <geometry>
-        <mesh filename="file://$(find turtlebot3_description)/meshes/wheels/right_tire.stl" scale="0.001 0.001 0.001"/>
+        <xacro:mesh mesh="wheels/right_tire.stl"/>
       </geometry>
       <material name="dark"/>
@@ -150,5 +149,5 @@
       <origin xyz="0 0 0.0" rpy="0 0 0"/>
       <geometry>
-        <mesh filename="file://$(find turtlebot3_description)/meshes/sensors/lds.stl" scale="0.001 0.001 0.001"/>
+        <xacro:mesh mesh="sensors/lds.stl"/>
       </geometry>
       <material name="dark"/>

Commit message: use Gazebo env hook to resolve package:// meshes

File: urdf/common_properties.xacro (robot description, xacro)
@@ -37,10 +37,5 @@
  </xacro:if>
  <xacro:macro name="mesh" params="mesh">
-   <xacro:if value="$(arg gazebo)">
-     <mesh filename="file://$(find turtlebot3_description)/meshes/${mesh}" scale="0.001 0.001 0.001"/>
-   </xacro:if>
-   <xacro:unless value="$(arg gazebo)">
      <mesh filename="package://turtlebot3_description/meshes/${mesh}" scale="0.001 0.001 0.001"/>
-   </xacro:unless>
  </xacro:macro>
 </robot>

Commit message: embed meshes

File: urdf/common_properties.xacro (robot description, xacro)
@@ -37,5 +37,5 @@
  </xacro:if>
  <xacro:macro name="mesh" params="mesh">
-     <mesh filename="package://turtlebot3_description/meshes/${mesh}" scale="0.001 0.001 0.001"/>
+     <mesh filename="package://turtlebot3_xacro/meshes/${mesh}" scale="0.001 0.001 0.001"/>
  </xacro:macro>
 </robot>
